Commit message: change tf tree to set base_footprint as root

File: pepper_description/urdf/pepper1.0_generated_urdf/pepper_legs.xacro (robot description, xacro)
@@ -5,7 +5,7 @@
 <robot xmlns:xacro="http://www.ros.org/wiki/xacro">
 	<joint name="HipRoll" type="revolute">
-		<parent link="torso"/>
-		<child link="Hip"/>
-		<origin rpy="0 0 0" xyz="2e-05 0 -0.139"/>
+		<child link="torso"/>
+		<parent link="Hip"/>
+		<origin rpy="0 0 0" xyz="-2e-05 0 0.139"/>
 		<axis xyz="1.0 0 0"/>
 		<limit effort="10.1884" lower="-0.514872" upper="0.514872" velocity="2.27032"/>
@@ -20,7 +20,7 @@
 	</link>
 	<joint name="HipPitch" type="revolute">
-		<parent link="Hip"/>
-		<child link="Pelvis"/>
-		<origin rpy="0 0 0" xyz="0 0 -0.079"/>
+		<child link="Hip"/>
+		<parent link="Pelvis"/>
+		<origin rpy="0 0 0" xyz="0 0 0.079"/>
 		<axis xyz="0 1.0 0"/>
 		<limit effort="19.787" lower="-1.03847" upper="1.03847" velocity="2.93276"/>
@@ -35,7 +35,7 @@
 	</link>
 	<joint name="KneePitch" type="revolute">
-		<parent link="Pelvis"/>
-		<child link="Tibia"/>
-		<origin rpy="0 0 0" xyz="0 0 -0.268"/>
+		<child link="Pelvis"/>
+		<parent link="Tibia"/>
+		<origin rpy="0 0 0" xyz="0 0 0.268"/>
 		<axis xyz="0 1.0 0"/>
 		<limit effort="27.702" lower="-0.514872" upper="0.514872" velocity="2.93276"/>
@@ -50,7 +50,7 @@
 	</link>
 	<joint name="base_footprint_joint" type="fixed">
-		<parent link="Tibia"/>
-		<child link="base_footprint"/>
-		<origin rpy="0 0 0" xyz="0 0 -0.334"/>
+		<parent link="base_footprint"/>
+		<child link="Tibia"/>
+		<origin rpy="0 0 0" xyz="0 0 0.334"/>
 	</joint>
 	<link name="base_footprint"/>

File: pepper_description/urdf/pepper1.0_generated_urdf/pepper_torso.xacro (robot description, xacro)
@@ -6,6 +6,6 @@
 	<link name="base_link"/>
 	<joint name="base_link_fixedjoint" type="fixed">
-		<parent link="base_link"/>
-		<child link="torso"/>
+		<child link="base_link"/>
+		<parent link="torso"/>
 		<origin rpy="0 0 0" xyz="0 0 0"/>
 		<axis xyz="0 0 0"/>
