Commit message: Revert "change mass and inertia to fix bugs"
This reverts commit 3094850ae5216c38a54decc6fa5b516d1a34e778.

File: pepper_description/urdf/pepper1.0_generated_urdf/pepper_fingers.xacro (robot description, xacro)
@@ -6,6 +6,6 @@
 	<link name="RFinger41_link">
 		<inertial>
-			<mass value="0.001" />
-			<inertia ixx="0" ixy="0" ixz="0" iyy="0" iyz="0" izz="0"/>
+			<mass value="2e-06"/>
+			<inertia ixx="1.1e-09" ixy="0" ixz="0" iyy="1.1e-09" iyz="0" izz="1.1e-09"/>
 		</inertial>
 		<xacro:insert_visu_RFinger41_link/>
@@ -20,6 +20,6 @@
 	<link name="LFinger42_link">
 		<inertial>
-			<mass value="0.001" />
-			<inertia ixx="0" ixy="0" ixz="0" iyy="0" iyz="0" izz="0"/>
+			<mass value="2e-06"/>
+			<inertia ixx="1.1e-09" ixy="0" ixz="0" iyy="1.1e-09" iyz="0" izz="1.1e-09"/>
 		</inertial>
 		<xacro:insert_visu_LFinger42_link/>
@@ -34,6 +34,6 @@
 	<link name="RFinger12_link">
 		<inertial>
-			<mass value="0.001" />
-			<inertia ixx="0" ixy="0" ixz="0" iyy="0" iyz="0" izz="0"/>
+			<mass value="2e-06"/>
+			<inertia ixx="1.1e-09" ixy="0" ixz="0" iyy="1.1e-09" iyz="0" izz="1.1e-09"/>
 		</inertial>
 		<xacro:insert_visu_RFinger12_link/>
@@ -48,6 +48,6 @@
 	<link name="LFinger33_link">
 		<inertial>
-			<mass value="0.001" />
-			<inertia ixx="0" ixy="0" ixz="0" iyy="0" iyz="0" izz="0"/>
+			<mass value="2e-06"/>
+			<inertia ixx="1.1e-09" ixy="0" ixz="0" iyy="1.1e-09" iyz="0" izz="1.1e-09"/>
 		</inertial>
 		<xacro:insert_visu_LFinger33_link/>
@@ -62,6 +62,6 @@
 	<link name="RFinger31_link">
 		<inertial>
-			<mass value="0.001" />
-			<inertia ixx="0" ixy="0" ixz="0" iyy="0" iyz="0" izz="0"/>
+			<mass value="2e-06"/>
+			<inertia ixx="1.1e-09" ixy="0" ixz="0" iyy="1.1e-09" iyz="0" izz="1.1e-09"/>
 		</inertial>
 		<xacro:insert_visu_RFinger31_link/>
@@ -76,6 +76,6 @@
 	<link name="LFinger21_link">
 		<inertial>
-			<mass value="0.001" />
-			<inertia ixx="0" ixy="0" ixz="0" iyy="0" iyz="0" izz="0"/>
+			<mass value="2e-06"/>
+			<inertia ixx="1.1e-09" ixy="0" ixz="0" iyy="1.1e-09" iyz="0" izz="1.1e-09"/>
 		</inertial>
 		<xacro:insert_visu_LFinger21_link/>
@@ -90,6 +90,6 @@
 	<link name="RFinger32_link">
 		<inertial>
-			<mass value="0.001" />
-			<inertia ixx="0" ixy="0" ixz="0" iyy="0" iyz="0" izz="0"/>
+			<mass value="2e-06"/>
+			<inertia ixx="1.1e-09" ixy="0" ixz="0" iyy="1.1e-09" iyz="0" izz="1.1e-09"/>
 		</inertial>
 		<xacro:insert_visu_RFinger32_link/>
@@ -104,6 +104,6 @@
 	<link name="LFinger13_link">
 		<inertial>
-			<mass value="0.001" />
-			<inertia ixx="0" ixy="0" ixz="0" iyy="0" iyz="0" izz="0"/>
+			<mass value="2e-06"/>
+			<inertia ixx="1.1e-09" ixy="0" ixz="0" iyy="1.1e-09" iyz="0" izz="1.1e-09"/>
 		</inertial>
 		<xacro:insert_visu_LFinger13_link/>
@@ -118,6 +118,6 @@
 	<link name="LFinger32_link">
 		<inertial>
-			<mass value="0.001" />
-			<inertia ixx="0" ixy="0" ixz="0" iyy="0" iyz="0" izz="0"/>
+			<mass value="2e-06"/>
+			<inertia ixx="1.1e-09" ixy="0" ixz="0" iyy="1.1e-09" iyz="0" izz="1.1e-09"/>
 		</inertial>
 		<xacro:insert_visu_LFinger32_link/>
@@ -132,6 +132,6 @@
 	<link name="LFinger11_link">
 		<inertial>
-			<mass value="0.001" />
-			<inertia ixx="0" ixy="0" ixz="0" iyy="0" iyz="0" izz="0"/>
+			<mass value="2e-06"/>
+			<inertia ixx="1.1e-09" ixy="0" ixz="0" iyy="1.1e-09" iyz="0" izz="1.1e-09"/>
 		</inertial>
 		<xacro:insert_visu_LFinger11_link/>
@@ -146,6 +146,6 @@
 	<link name="RFinger22_link">
 		<inertial>
-			<mass value="0.001" />
-			<inertia ixx="0" ixy="0" ixz="0" iyy="0" iyz="0" izz="0"/>
+			<mass value="2e-06"/>
+			<inertia ixx="1.1e-09" ixy="0" ixz="0" iyy="1.1e-09" iyz="0" izz="1.1e-09"/>
 		</inertial>
 		<xacro:insert_visu_RFinger22_link/>
@@ -160,6 +160,6 @@
 	<link name="RFinger13_link">
 		<inertial>
-			<mass value="0.001" />
-			<inertia ixx="0" ixy="0" ixz="0" iyy="0" iyz="0" izz="0"/>
+			<mass value="2e-06"/>
+			<inertia ixx="1.1e-09" ixy="0" ixz="0" iyy="1.1e-09" iyz="0" izz="1.1e-09"/>
 		</inertial>
 		<xacro:insert_visu_RFinger13_link/>
@@ -174,6 +174,6 @@
 	<link name="LFinger22_link">
 		<inertial>
-			<mass value="0.001" />
-			<inertia ixx="0" ixy="0" ixz="0" iyy="0" iyz="0" izz="0"/>
+			<mass value="2e-06"/>
+			<inertia ixx="1.1e-09" ixy="0" ixz="0" iyy="1.1e-09" iyz="0" izz="1.1e-09"/>
 		</inertial>
 		<xacro:insert_visu_LFinger22_link/>
@@ -188,6 +188,6 @@
 	<link name="RFinger21_link">
 		<inertial>
-			<mass value="0.001" />
-			<inertia ixx="0" ixy="0" ixz="0" iyy="0" iyz="0" izz="0"/>
+			<mass value="2e-06"/>
+			<inertia ixx="1.1e-09" ixy="0" ixz="0" iyy="1.1e-09" iyz="0" izz="1.1e-09"/>
 		</inertial>
 		<xacro:insert_visu_RFinger21_link/>
@@ -202,6 +202,6 @@
 	<link name="LFinger41_link">
 		<inertial>
-			<mass value="0.001" />
-			<inertia ixx="0" ixy="0" ixz="0" iyy="0" iyz="0" izz="0"/>
+			<mass value="2e-06"/>
+			<inertia ixx="1.1e-09" ixy="0" ixz="0" iyy="1.1e-09" iyz="0" izz="1.1e-09"/>
 		</inertial>
 		<xacro:insert_visu_LFinger41_link/>
@@ -216,6 +216,6 @@
 	<link name="LFinger12_link">
 		<inertial>
-			<mass value="0.001" />
-			<inertia ixx="0" ixy="0" ixz="0" iyy="0" iyz="0" izz="0"/>
+			<mass value="2e-06"/>
+			<inertia ixx="1.1e-09" ixy="0" ixz="0" iyy="1.1e-09" iyz="0" izz="1.1e-09"/>
 		</inertial>
 		<xacro:insert_visu_LFinger12_link/>
@@ -230,6 +230,6 @@
 	<link name="RFinger23_link">
 		<inertial>
-			<mass value="0.001" />
-			<inertia ixx="0" ixy="0" ixz="0" iyy="0" iyz="0" izz="0"/>
+			<mass value="2e-06"/>
+			<inertia ixx="1.1e-09" ixy="0" ixz="0" iyy="1.1e-09" iyz="0" izz="1.1e-09"/>
 		</inertial>
 		<xacro:insert_visu_RFinger23_link/>
@@ -244,6 +244,6 @@
 	<link name="RFinger11_link">
 		<inertial>
-			<mass value="0.001" />
-			<inertia ixx="0" ixy="0" ixz="0" iyy="0" iyz="0" izz="0"/>
+			<mass value="2e-06"/>
+			<inertia ixx="1.1e-09" ixy="0" ixz="0" iyy="1.1e-09" iyz="0" izz="1.1e-09"/>
 		</inertial>
 		<xacro:insert_visu_RFinger11_link/>
@@ -258,6 +258,6 @@
 	<link name="LFinger23_link">
 		<inertial>
-			<mass value="0.001" />
-			<inertia ixx="0" ixy="0" ixz="0" iyy="0" iyz="0" izz="0"/>
+			<mass value="2e-06"/>
+			<inertia ixx="1.1e-09" ixy="0" ixz="0" iyy="1.1e-09" iyz="0" izz="1.1e-09"/>
 		</inertial>
 		<xacro:insert_visu_LFinger23_link/>
@@ -272,6 +272,6 @@
 	<link name="LFinger43_link">
 		<inertial>
-			<mass value="0.001" />
-			<inertia ixx="0" ixy="0" ixz="0" iyy="0" iyz="0" izz="0"/>
+			<mass value="2e-06"/>
+			<inertia ixx="1.1e-09" ixy="0" ixz="0" iyy="1.1e-09" iyz="0" izz="1.1e-09"/>
 		</inertial>
 		<xacro:insert_visu_LFinger43_link/>
@@ -286,6 +286,6 @@
 	<link name="RFinger43_link">
 		<inertial>
-			<mass value="0.001" />
-			<inertia ixx="0" ixy="0" ixz="0" iyy="0" iyz="0" izz="0"/>
+			<mass value="2e-06"/>
+			<inertia ixx="1.1e-09" ixy="0" ixz="0" iyy="1.1e-09" iyz="0" izz="1.1e-09"/>
 		</inertial>
 		<xacro:insert_visu_RFinger43_link/>
@@ -300,6 +300,6 @@
 	<link name="RFinger42_link">
 		<inertial>
-			<mass value="0.001" />
-			<inertia ixx="0" ixy="0" ixz="0" iyy="0" iyz="0" izz="0"/>
+			<mass value="2e-06"/>
+			<inertia ixx="1.1e-09" ixy="0" ixz="0" iyy="1.1e-09" iyz="0" izz="1.1e-09"/>
 		</inertial>
 		<xacro:insert_visu_RFinger42_link/>
@@ -314,6 +314,6 @@
 	<link name="LFinger31_link">
 		<inertial>
-			<mass value="0.001" />
-			<inertia ixx="0" ixy="0" ixz="0" iyy="0" iyz="0" izz="0"/>
+			<mass value="2e-06"/>
+			<inertia ixx="1.1e-09" ixy="0" ixz="0" iyy="1.1e-09" iyz="0" izz="1.1e-09"/>
 		</inertial>
 		<xacro:insert_visu_LFinger31_link/>
@@ -328,6 +328,6 @@
 	<link name="RFinger33_link">
 		<inertial>
-			<mass value="0.001" />
-			<inertia ixx="0" ixy="0" ixz="0" iyy="0" iyz="0" izz="0"/>
+			<mass value="2e-06"/>
+			<inertia ixx="1.1e-09" ixy="0" ixz="0" iyy="1.1e-09" iyz="0" izz="1.1e-09"/>
 		</inertial>
 		<xacro:insert_visu_RFinger33_link/>
@@ -342,6 +342,6 @@
 	<link name="LThumb1_link">
 		<inertial>
-			<mass value="0.001" />
-			<inertia ixx="0" ixy="0" ixz="0" iyy="0" iyz="0" izz="0"/>
+			<mass value="2e-06"/>
+			<inertia ixx="1.1e-09" ixy="0" ixz="0" iyy="1.1e-09" iyz="0" izz="1.1e-09"/>
 		</inertial>
 		<xacro:insert_visu_LThumb1_link/>
@@ -356,6 +356,6 @@
 	<link name="RThumb2_link">
 		<inertial>
-			<mass value="0.001" />
-			<inertia ixx="0" ixy="0" ixz="0" iyy="0" iyz="0" izz="0"/>
+			<mass value="2e-06"/>
+			<inertia ixx="1.1e-09" ixy="0" ixz="0" iyy="1.1e-09" iyz="0" izz="1.1e-09"/>
 		</inertial>
 		<xacro:insert_visu_RThumb2_link/>
@@ -370,6 +370,6 @@
 	<link name="RThumb1_link">
 		<inertial>
-			<mass value="0.001" />
-			<inertia ixx="0" ixy="0" ixz="0" iyy="0" iyz="0" izz="0"/>
+			<mass value="2e-06"/>
+			<inertia ixx="1.1e-09" ixy="0" ixz="0" iyy="1.1e-09" iyz="0" izz="1.1e-09"/>
 		</inertial>
 		<xacro:insert_visu_RThumb1_link/>
@@ -384,6 +384,6 @@
 	<link name="LThumb2_link">
 		<inertial>
-			<mass value="0.001" />
-			<inertia ixx="0" ixy="0" ixz="0" iyy="0" iyz="0" izz="0"/>
+			<mass value="2e-06"/>
+			<inertia ixx="1.1e-09" ixy="0" ixz="0" iyy="1.1e-09" iyz="0" izz="1.1e-09"/>
 		</inertial>
 		<xacro:insert_visu_LThumb2_link/>

Commit message: change mass and inertia to fix bugs

File: pepper_description/urdf/pepper1.0_generated_urdf/pepper_fingers.xacro (robot description, xacro)
@@ -6,6 +6,6 @@
 	<link name="RFinger41_link">
 		<inertial>
-			<mass value="2e-06"/>
-			<inertia ixx="1.1e-09" ixy="0" ixz="0" iyy="1.1e-09" iyz="0" izz="1.1e-09"/>
+			<mass value="0.001" />
+			<inertia ixx="0" ixy="0" ixz="0" iyy="0" iyz="0" izz="0"/>
 		</inertial>
 		<xacro:insert_visu_RFinger41_link/>
@@ -20,6 +20,6 @@
 	<link name="LFinger42_link">
 		<inertial>
-			<mass value="2e-06"/>
-			<inertia ixx="1.1e-09" ixy="0" ixz="0" iyy="1.1e-09" iyz="0" izz="1.1e-09"/>
+			<mass value="0.001" />
+			<inertia ixx="0" ixy="0" ixz="0" iyy="0" iyz="0" izz="0"/>
 		</inertial>
 		<xacro:insert_visu_LFinger42_link/>
@@ -34,6 +34,6 @@
 	<link name="RFinger12_link">
 		<inertial>
-			<mass value="2e-06"/>
-			<inertia ixx="1.1e-09" ixy="0" ixz="0" iyy="1.1e-09" iyz="0" izz="1.1e-09"/>
+			<mass value="0.001" />
+			<inertia ixx="0" ixy="0" ixz="0" iyy="0" iyz="0" izz="0"/>
 		</inertial>
 		<xacro:insert_visu_RFinger12_link/>
@@ -48,6 +48,6 @@
 	<link name="LFinger33_link">
 		<inertial>
-			<mass value="2e-06"/>
-			<inertia ixx="1.1e-09" ixy="0" ixz="0" iyy="1.1e-09" iyz="0" izz="1.1e-09"/>
+			<mass value="0.001" />
+			<inertia ixx="0" ixy="0" ixz="0" iyy="0" iyz="0" izz="0"/>
 		</inertial>
 		<xacro:insert_visu_LFinger33_link/>
@@ -62,6 +62,6 @@
 	<link name="RFinger31_link">
 		<inertial>
-			<mass value="2e-06"/>
-			<inertia ixx="1.1e-09" ixy="0" ixz="0" iyy="1.1e-09" iyz="0" izz="1.1e-09"/>
+			<mass value="0.001" />
+			<inertia ixx="0" ixy="0" ixz="0" iyy="0" iyz="0" izz="0"/>
 		</inertial>
 		<xacro:insert_visu_RFinger31_link/>
@@ -76,6 +76,6 @@
 	<link name="LFinger21_link">
 		<inertial>
-			<mass value="2e-06"/>
-			<inertia ixx="1.1e-09" ixy="0" ixz="0" iyy="1.1e-09" iyz="0" izz="1.1e-09"/>
+			<mass value="0.001" />
+			<inertia ixx="0" ixy="0" ixz="0" iyy="0" iyz="0" izz="0"/>
 		</inertial>
 		<xacro:insert_visu_LFinger21_link/>
@@ -90,6 +90,6 @@
 	<link name="RFinger32_link">
 		<inertial>
-			<mass value="2e-06"/>
-			<inertia ixx="1.1e-09" ixy="0" ixz="0" iyy="1.1e-09" iyz="0" izz="1.1e-09"/>
+			<mass value="0.001" />
+			<inertia ixx="0" ixy="0" ixz="0" iyy="0" iyz="0" izz="0"/>
 		</inertial>
 		<xacro:insert_visu_RFinger32_link/>
@@ -104,6 +104,6 @@
 	<link name="LFinger13_link">
 		<inertial>
-			<mass value="2e-06"/>
-			<inertia ixx="1.1e-09" ixy="0" ixz="0" iyy="1.1e-09" iyz="0" izz="1.1e-09"/>
+			<mass value="0.001" />
+			<inertia ixx="0" ixy="0" ixz="0" iyy="0" iyz="0" izz="0"/>
 		</inertial>
 		<xacro:insert_visu_LFinger13_link/>
@@ -118,6 +118,6 @@
 	<link name="LFinger32_link">
 		<inertial>
-			<mass value="2e-06"/>
-			<inertia ixx="1.1e-09" ixy="0" ixz="0" iyy="1.1e-09" iyz="0" izz="1.1e-09"/>
+			<mass value="0.001" />
+			<inertia ixx="0" ixy="0" ixz="0" iyy="0" iyz="0" izz="0"/>
 		</inertial>
 		<xacro:insert_visu_LFinger32_link/>
@@ -132,6 +132,6 @@
 	<link name="LFinger11_link">
 		<inertial>
-			<mass value="2e-06"/>
-			<inertia ixx="1.1e-09" ixy="0" ixz="0" iyy="1.1e-09" iyz="0" izz="1.1e-09"/>
+			<mass value="0.001" />
+			<inertia ixx="0" ixy="0" ixz="0" iyy="0" iyz="0" izz="0"/>
 		</inertial>
 		<xacro:insert_visu_LFinger11_link/>
@@ -146,6 +146,6 @@
 	<link name="RFinger22_link">
 		<inertial>
-			<mass value="2e-06"/>
-			<inertia ixx="1.1e-09" ixy="0" ixz="0" iyy="1.1e-09" iyz="0" izz="1.1e-09"/>
+			<mass value="0.001" />
+			<inertia ixx="0" ixy="0" ixz="0" iyy="0" iyz="0" izz="0"/>
 		</inertial>
 		<xacro:insert_visu_RFinger22_link/>
@@ -160,6 +160,6 @@
 	<link name="RFinger13_link">
 		<inertial>
-			<mass value="2e-06"/>
-			<inertia ixx="1.1e-09" ixy="0" ixz="0" iyy="1.1e-09" iyz="0" izz="1.1e-09"/>
+			<mass value="0.001" />
+			<inertia ixx="0" ixy="0" ixz="0" iyy="0" iyz="0" izz="0"/>
 		</inertial>
 		<xacro:insert_visu_RFinger13_link/>
@@ -174,6 +174,6 @@
 	<link name="LFinger22_link">
 		<inertial>
-			<mass value="2e-06"/>
-			<inertia ixx="1.1e-09" ixy="0" ixz="0" iyy="1.1e-09" iyz="0" izz="1.1e-09"/>
+			<mass value="0.001" />
+			<inertia ixx="0" ixy="0" ixz="0" iyy="0" iyz="0" izz="0"/>
 		</inertial>
 		<xacro:insert_visu_LFinger22_link/>
@@ -188,6 +188,6 @@
 	<link name="RFinger21_link">
 		<inertial>
-			<mass value="2e-06"/>
-			<inertia ixx="1.1e-09" ixy="0" ixz="0" iyy="1.1e-09" iyz="0" izz="1.1e-09"/>
+			<mass value="0.001" />
+			<inertia ixx="0" ixy="0" ixz="0" iyy="0" iyz="0" izz="0"/>
 		</inertial>
 		<xacro:insert_visu_RFinger21_link/>
@@ -202,6 +202,6 @@
 	<link name="LFinger41_link">
 		<inertial>
-			<mass value="2e-06"/>
-			<inertia ixx="1.1e-09" ixy="0" ixz="0" iyy="1.1e-09" iyz="0" izz="1.1e-09"/>
+			<mass value="0.001" />
+			<inertia ixx="0" ixy="0" ixz="0" iyy="0" iyz="0" izz="0"/>
 		</inertial>
 		<xacro:insert_visu_LFinger41_link/>
@@ -216,6 +216,6 @@
 	<link name="LFinger12_link">
 		<inertial>
-			<mass value="2e-06"/>
-			<inertia ixx="1.1e-09" ixy="0" ixz="0" iyy="1.1e-09" iyz="0" izz="1.1e-09"/>
+			<mass value="0.001" />
+			<inertia ixx="0" ixy="0" ixz="0" iyy="0" iyz="0" izz="0"/>
 		</inertial>
 		<xacro:insert_visu_LFinger12_link/>
@@ -230,6 +230,6 @@
 	<link name="RFinger23_link">
 		<inertial>
-			<mass value="2e-06"/>
-			<inertia ixx="1.1e-09" ixy="0" ixz="0" iyy="1.1e-09" iyz="0" izz="1.1e-09"/>
+			<mass value="0.001" />
+			<inertia ixx="0" ixy="0" ixz="0" iyy="0" iyz="0" izz="0"/>
 		</inertial>
 		<xacro:insert_visu_RFinger23_link/>
@@ -244,6 +244,6 @@
 	<link name="RFinger11_link">
 		<inertial>
-			<mass value="2e-06"/>
-			<inertia ixx="1.1e-09" ixy="0" ixz="0" iyy="1.1e-09" iyz="0" izz="1.1e-09"/>
+			<mass value="0.001" />
+			<inertia ixx="0" ixy="0" ixz="0" iyy="0" iyz="0" izz="0"/>
 		</inertial>
 		<xacro:insert_visu_RFinger11_link/>
@@ -258,6 +258,6 @@
 	<link name="LFinger23_link">
 		<inertial>
-			<mass value="2e-06"/>
-			<inertia ixx="1.1e-09" ixy="0" ixz="0" iyy="1.1e-09" iyz="0" izz="1.1e-09"/>
+			<mass value="0.001" />
+			<inertia ixx="0" ixy="0" ixz="0" iyy="0" iyz="0" izz="0"/>
 		</inertial>
 		<xacro:insert_visu_LFinger23_link/>
@@ -272,6 +272,6 @@
 	<link name="LFinger43_link">
 		<inertial>
-			<mass value="2e-06"/>
-			<inertia ixx="1.1e-09" ixy="0" ixz="0" iyy="1.1e-09" iyz="0" izz="1.1e-09"/>
+			<mass value="0.001" />
+			<inertia ixx="0" ixy="0" ixz="0" iyy="0" iyz="0" izz="0"/>
 		</inertial>
 		<xacro:insert_visu_LFinger43_link/>
@@ -286,6 +286,6 @@
 	<link name="RFinger43_link">
 		<inertial>
-			<mass value="2e-06"/>
-			<inertia ixx="1.1e-09" ixy="0" ixz="0" iyy="1.1e-09" iyz="0" izz="1.1e-09"/>
+			<mass value="0.001" />
+			<inertia ixx="0" ixy="0" ixz="0" iyy="0" iyz="0" izz="0"/>
 		</inertial>
 		<xacro:insert_visu_RFinger43_link/>
@@ -300,6 +300,6 @@
 	<link name="RFinger42_link">
 		<inertial>
-			<mass value="2e-06"/>
-			<inertia ixx="1.1e-09" ixy="0" ixz="0" iyy="1.1e-09" iyz="0" izz="1.1e-09"/>
+			<mass value="0.001" />
+			<inertia ixx="0" ixy="0" ixz="0" iyy="0" iyz="0" izz="0"/>
 		</inertial>
 		<xacro:insert_visu_RFinger42_link/>
@@ -314,6 +314,6 @@
 	<link name="LFinger31_link">
 		<inertial>
-			<mass value="2e-06"/>
-			<inertia ixx="1.1e-09" ixy="0" ixz="0" iyy="1.1e-09" iyz="0" izz="1.1e-09"/>
+			<mass value="0.001" />
+			<inertia ixx="0" ixy="0" ixz="0" iyy="0" iyz="0" izz="0"/>
 		</inertial>
 		<xacro:insert_visu_LFinger31_link/>
@@ -328,6 +328,6 @@
 	<link name="RFinger33_link">
 		<inertial>
-			<mass value="2e-06"/>
-			<inertia ixx="1.1e-09" ixy="0" ixz="0" iyy="1.1e-09" iyz="0" izz="1.1e-09"/>
+			<mass value="0.001" />
+			<inertia ixx="0" ixy="0" ixz="0" iyy="0" iyz="0" izz="0"/>
 		</inertial>
 		<xacro:insert_visu_RFinger33_link/>
@@ -342,6 +342,6 @@
 	<link name="LThumb1_link">
 		<inertial>
-			<mass value="2e-06"/>
-			<inertia ixx="1.1e-09" ixy="0" ixz="0" iyy="1.1e-09" iyz="0" izz="1.1e-09"/>
+			<mass value="0.001" />
+			<inertia ixx="0" ixy="0" ixz="0" iyy="0" iyz="0" izz="0"/>
 		</inertial>
 		<xacro:insert_visu_LThumb1_link/>
@@ -356,6 +356,6 @@
 	<link name="RThumb2_link">
 		<inertial>
-			<mass value="2e-06"/>
-			<inertia ixx="1.1e-09" ixy="0" ixz="0" iyy="1.1e-09" iyz="0" izz="1.1e-09"/>
+			<mass value="0.001" />
+			<inertia ixx="0" ixy="0" ixz="0" iyy="0" iyz="0" izz="0"/>
 		</inertial>
 		<xacro:insert_visu_RThumb2_link/>
@@ -370,6 +370,6 @@
 	<link name="RThumb1_link">
 		<inertial>
-			<mass value="2e-06"/>
-			<inertia ixx="1.1e-09" ixy="0" ixz="0" iyy="1.1e-09" iyz="0" izz="1.1e-09"/>
+			<mass value="0.001" />
+			<inertia ixx="0" ixy="0" ixz="0" iyy="0" iyz="0" izz="0"/>
 		</inertial>
 		<xacro:insert_visu_RThumb1_link/>
@@ -384,6 +384,6 @@
 	<link name="LThumb2_link">
 		<inertial>
-			<mass value="2e-06"/>
-			<inertia ixx="1.1e-09" ixy="0" ixz="0" iyy="1.1e-09" iyz="0" izz="1.1e-09"/>
+			<mass value="0.001" />
+			<inertia ixx="0" ixy="0" ixz="0" iyy="0" iyz="0" izz="0"/>
 		</inertial>
 		<xacro:insert_visu_LThumb2_link/>
