Commit message: remove some fingers
Some fingers rotate infinity

File: pepper_description/urdf/pepper1.0_generated_urdf/pepper_fingers.xacro (robot description, xacro)
@@ -6,6 +6,6 @@
 	<link name="RFinger41_link">
 		<inertial>
-			<mass value="2e-06"/>
-			<inertia ixx="1.1e-09" ixy="0" ixz="0" iyy="1.1e-09" iyz="0" izz="1.1e-09"/>
+			<mass value="0"/>
+			<inertia ixx="0" ixy="0" ixz="0" iyy="0" iyz="0" izz="0"/>
 		</inertial>
 		<xacro:insert_visu_RFinger41_link/>
@@ -20,6 +20,6 @@
 	<link name="LFinger42_link">
 		<inertial>
-			<mass value="2e-06"/>
-			<inertia ixx="1.1e-09" ixy="0" ixz="0" iyy="1.1e-09" iyz="0" izz="1.1e-09"/>
+			<mass value="0"/>
+			<inertia ixx="0" ixy="0" ixz="0" iyy="0" iyz="0" izz="0"/>
 		</inertial>
 		<xacro:insert_visu_LFinger42_link/>
@@ -34,6 +34,6 @@
 	<link name="RFinger12_link">
 		<inertial>
-			<mass value="2e-06"/>
-			<inertia ixx="1.1e-09" ixy="0" ixz="0" iyy="1.1e-09" iyz="0" izz="1.1e-09"/>
+			<mass value="0.001"/>
+			<inertia ixx="0" ixy="0" ixz="0" iyy="0" iyz="0" izz="0"/>
 		</inertial>
 		<xacro:insert_visu_RFinger12_link/>
@@ -48,6 +48,6 @@
 	<link name="LFinger33_link">
 		<inertial>
-			<mass value="2e-06"/>
-			<inertia ixx="1.1e-09" ixy="0" ixz="0" iyy="1.1e-09" iyz="0" izz="1.1e-09"/>
+			<mass value="0"/>
+			<inertia ixx="0" ixy="0" ixz="0" iyy="0" iyz="0" izz="0"/>
 		</inertial>
 		<xacro:insert_visu_LFinger33_link/>
@@ -62,6 +62,6 @@
 	<link name="RFinger31_link">
 		<inertial>
-			<mass value="2e-06"/>
-			<inertia ixx="1.1e-09" ixy="0" ixz="0" iyy="1.1e-09" iyz="0" izz="1.1e-09"/>
+			<mass value="0"/>
+			<inertia ixx="0" ixy="0" ixz="0" iyy="0" iyz="0" izz="0"/>
 		</inertial>
 		<xacro:insert_visu_RFinger31_link/>
@@ -76,6 +76,6 @@
 	<link name="LFinger21_link">
 		<inertial>
-			<mass value="2e-06"/>
-			<inertia ixx="1.1e-09" ixy="0" ixz="0" iyy="1.1e-09" iyz="0" izz="1.1e-09"/>
+			<mass value="0"/>
+			<inertia ixx="0" ixy="0" ixz="0" iyy="0" iyz="0" izz="0"/>
 		</inertial>
 		<xacro:insert_visu_LFinger21_link/>
@@ -90,6 +90,6 @@
 	<link name="RFinger32_link">
 		<inertial>
-			<mass value="2e-06"/>
-			<inertia ixx="1.1e-09" ixy="0" ixz="0" iyy="1.1e-09" iyz="0" izz="1.1e-09"/>
+			<mass value="0"/>
+			<inertia ixx="0" ixy="0" ixz="0" iyy="0" iyz="0" izz="0"/>
 		</inertial>
 		<xacro:insert_visu_RFinger32_link/>
@@ -104,6 +104,6 @@
 	<link name="LFinger13_link">
 		<inertial>
-			<mass value="2e-06"/>
-			<inertia ixx="1.1e-09" ixy="0" ixz="0" iyy="1.1e-09" iyz="0" izz="1.1e-09"/>
+			<mass value="0.001"/>
+			<inertia ixx="0" ixy="0" ixz="0" iyy="0" iyz="0" izz="0"/>
 		</inertial>
 		<xacro:insert_visu_LFinger13_link/>
@@ -118,6 +118,6 @@
 	<link name="LFinger32_link">
 		<inertial>
-			<mass value="2e-06"/>
-			<inertia ixx="1.1e-09" ixy="0" ixz="0" iyy="1.1e-09" iyz="0" izz="1.1e-09"/>
+			<mass value="0"/>
+			<inertia ixx="0" ixy="0" ixz="0" iyy="0" iyz="0" izz="0"/>
 		</inertial>
 		<xacro:insert_visu_LFinger32_link/>
@@ -132,6 +132,6 @@
 	<link name="LFinger11_link">
 		<inertial>
-			<mass value="2e-06"/>
-			<inertia ixx="1.1e-09" ixy="0" ixz="0" iyy="1.1e-09" iyz="0" izz="1.1e-09"/>
+			<mass value="0.001"/>
+			<inertia ixx="0" ixy="0" ixz="0" iyy="0" iyz="0" izz="0"/>
 		</inertial>
 		<xacro:insert_visu_LFinger11_link/>
@@ -146,6 +146,6 @@
 	<link name="RFinger22_link">
 		<inertial>
-			<mass value="2e-06"/>
-			<inertia ixx="1.1e-09" ixy="0" ixz="0" iyy="1.1e-09" iyz="0" izz="1.1e-09"/>
+			<mass value="0"/>
+			<inertia ixx="0" ixy="0" ixz="0" iyy="0" iyz="0" izz="0"/>
 		</inertial>
 		<xacro:insert_visu_RFinger22_link/>
@@ -160,6 +160,6 @@
 	<link name="RFinger13_link">
 		<inertial>
-			<mass value="2e-06"/>
-			<inertia ixx="1.1e-09" ixy="0" ixz="0" iyy="1.1e-09" iyz="0" izz="1.1e-09"/>
+			<mass value="0.001"/>
+			<inertia ixx="0" ixy="0" ixz="0" iyy="0" iyz="0" izz="0"/>
 		</inertial>
 		<xacro:insert_visu_RFinger13_link/>
@@ -174,6 +174,6 @@
 	<link name="LFinger22_link">
 		<inertial>
-			<mass value="2e-06"/>
-			<inertia ixx="1.1e-09" ixy="0" ixz="0" iyy="1.1e-09" iyz="0" izz="1.1e-09"/>
+			<mass value="0"/>
+			<inertia ixx="0" ixy="0" ixz="0" iyy="0" iyz="0" izz="0"/>
 		</inertial>
 		<xacro:insert_visu_LFinger22_link/>
@@ -188,6 +188,6 @@
 	<link name="RFinger21_link">
 		<inertial>
-			<mass value="2e-06"/>
-			<inertia ixx="1.1e-09" ixy="0" ixz="0" iyy="1.1e-09" iyz="0" izz="1.1e-09"/>
+			<mass value="0"/>
+			<inertia ixx="0" ixy="0" ixz="0" iyy="0" iyz="0" izz="0"/>
 		</inertial>
 		<xacro:insert_visu_RFinger21_link/>
@@ -202,6 +202,6 @@
 	<link name="LFinger41_link">
 		<inertial>
-			<mass value="2e-06"/>
-			<inertia ixx="1.1e-09" ixy="0" ixz="0" iyy="1.1e-09" iyz="0" izz="1.1e-09"/>
+			<mass value="0"/>
+			<inertia ixx="0" ixy="0" ixz="0" iyy="0" iyz="0" izz="0"/>
 		</inertial>
 		<xacro:insert_visu_LFinger41_link/>
@@ -216,6 +216,6 @@
 	<link name="LFinger12_link">
 		<inertial>
-			<mass value="2e-06"/>
-			<inertia ixx="1.1e-09" ixy="0" ixz="0" iyy="1.1e-09" iyz="0" izz="1.1e-09"/>
+			<mass value="0.001"/>
+			<inertia ixx="0" ixy="0" ixz="0" iyy="0" iyz="0" izz="0"/>
 		</inertial>
 		<xacro:insert_visu_LFinger12_link/>
@@ -230,6 +230,6 @@
 	<link name="RFinger23_link">
 		<inertial>
-			<mass value="2e-06"/>
-			<inertia ixx="1.1e-09" ixy="0" ixz="0" iyy="1.1e-09" iyz="0" izz="1.1e-09"/>
+			<mass value="0"/>
+			<inertia ixx="0" ixy="0" ixz="0" iyy="0" iyz="0" izz="0"/>
 		</inertial>
 		<xacro:insert_visu_RFinger23_link/>
@@ -244,6 +244,6 @@
 	<link name="RFinger11_link">
 		<inertial>
-			<mass value="2e-06"/>
-			<inertia ixx="1.1e-09" ixy="0" ixz="0" iyy="1.1e-09" iyz="0" izz="1.1e-09"/>
+			<mass value="0.001"/>
+			<inertia ixx="0" ixy="0" ixz="0" iyy="0" iyz="0" izz="0"/>
 		</inertial>
 		<xacro:insert_visu_RFinger11_link/>
@@ -258,6 +258,6 @@
 	<link name="LFinger23_link">
 		<inertial>
-			<mass value="2e-06"/>
-			<inertia ixx="1.1e-09" ixy="0" ixz="0" iyy="1.1e-09" iyz="0" izz="1.1e-09"/>
+			<mass value="0"/>
+			<inertia ixx="0" ixy="0" ixz="0" iyy="0" iyz="0" izz="0"/>
 		</inertial>
 		<xacro:insert_visu_LFinger23_link/>
@@ -272,6 +272,6 @@
 	<link name="LFinger43_link">
 		<inertial>
-			<mass value="2e-06"/>
-			<inertia ixx="1.1e-09" ixy="0" ixz="0" iyy="1.1e-09" iyz="0" izz="1.1e-09"/>
+			<mass value="0"/>
+			<inertia ixx="0" ixy="0" ixz="0" iyy="0" iyz="0" izz="0"/>
 		</inertial>
 		<xacro:insert_visu_LFinger43_link/>
@@ -286,6 +286,6 @@
 	<link name="RFinger43_link">
 		<inertial>
-			<mass value="2e-06"/>
-			<inertia ixx="1.1e-09" ixy="0" ixz="0" iyy="1.1e-09" iyz="0" izz="1.1e-09"/>
+			<mass value="0"/>
+			<inertia ixx="0" ixy="0" ixz="0" iyy="0" iyz="0" izz="0"/>
 		</inertial>
 		<xacro:insert_visu_RFinger43_link/>
@@ -300,6 +300,6 @@
 	<link name="RFinger42_link">
 		<inertial>
-			<mass value="2e-06"/>
-			<inertia ixx="1.1e-09" ixy="0" ixz="0" iyy="1.1e-09" iyz="0" izz="1.1e-09"/>
+			<mass value="0"/>
+			<inertia ixx="0" ixy="0" ixz="0" iyy="0" iyz="0" izz="0"/>
 		</inertial>
 		<xacro:insert_visu_RFinger42_link/>
@@ -314,6 +314,6 @@
 	<link name="LFinger31_link">
 		<inertial>
-			<mass value="2e-06"/>
-			<inertia ixx="1.1e-09" ixy="0" ixz="0" iyy="1.1e-09" iyz="0" izz="1.1e-09"/>
+			<mass value="0"/>
+			<inertia ixx="0" ixy="0" ixz="0" iyy="0" iyz="0" izz="0"/>
 		</inertial>
 		<xacro:insert_visu_LFinger31_link/>
@@ -328,6 +328,6 @@
 	<link name="RFinger33_link">
 		<inertial>
-			<mass value="2e-06"/>
-			<inertia ixx="1.1e-09" ixy="0" ixz="0" iyy="1.1e-09" iyz="0" izz="1.1e-09"/>
+			<mass value="0"/>
+			<inertia ixx="0" ixy="0" ixz="0" iyy="0" iyz="0" izz="0"/>
 		</inertial>
 		<xacro:insert_visu_RFinger33_link/>
@@ -342,6 +342,6 @@
 	<link name="LThumb1_link">
 		<inertial>
-			<mass value="2e-06"/>
-			<inertia ixx="1.1e-09" ixy="0" ixz="0" iyy="1.1e-09" iyz="0" izz="1.1e-09"/>
+			<mass value="0.001"/>
+			<inertia ixx="0" ixy="0" ixz="0" iyy="0" iyz="0" izz="0"/>
 		</inertial>
 		<xacro:insert_visu_LThumb1_link/>
@@ -356,6 +356,6 @@
 	<link name="RThumb2_link">
 		<inertial>
-			<mass value="2e-06"/>
-			<inertia ixx="1.1e-09" ixy="0" ixz="0" iyy="1.1e-09" iyz="0" izz="1.1e-09"/>
+			<mass value="0.001"/>
+			<inertia ixx="0" ixy="0" ixz="0" iyy="0" iyz="0" izz="0"/>
 		</inertial>
 		<xacro:insert_visu_RThumb2_link/>
@@ -370,6 +370,6 @@
 	<link name="RThumb1_link">
 		<inertial>
-			<mass value="2e-06"/>
-			<inertia ixx="1.1e-09" ixy="0" ixz="0" iyy="1.1e-09" iyz="0" izz="1.1e-09"/>
+			<mass value="0.001"/>
+			<inertia ixx="0" ixy="0" ixz="0" iyy="0" iyz="0" izz="0"/>
 		</inertial>
 		<xacro:insert_visu_RThumb1_link/>
@@ -384,6 +384,6 @@
 	<link name="LThumb2_link">
 		<inertial>
-			<mass value="2e-06"/>
-			<inertia ixx="1.1e-09" ixy="0" ixz="0" iyy="1.1e-09" iyz="0" izz="1.1e-09"/>
+			<mass value="0.001"/>
+			<inertia ixx="0" ixy="0" ixz="0" iyy="0" iyz="0" izz="0"/>
 		</inertial>
 		<xacro:insert_visu_LThumb2_link/>

Commit message: change finger joints to fixed

File: pepper_description/urdf/pepper1.0_generated_urdf/pepper_fingers.xacro (robot description, xacro)
@@ -6,10 +6,10 @@
 	<link name="RFinger41_link">
 		<inertial>
-			<mass value="0"/>
+			<mass value="0.001"/>
 			<inertia ixx="0" ixy="0" ixz="0" iyy="0" iyz="0" izz="0"/>
 		</inertial>
 		<xacro:insert_visu_RFinger41_link/>
 	</link>
-	<joint name="RFinger41" type="continuous">
+	<joint name="RFinger41" type="fixed">
 		<parent link="r_wrist"/>
 		<child link="RFinger41_link"/>
@@ -20,10 +20,10 @@
 	<link name="LFinger42_link">
 		<inertial>
-			<mass value="0"/>
+			<mass value="0.001"/>
 			<inertia ixx="0" ixy="0" ixz="0" iyy="0" iyz="0" izz="0"/>
 		</inertial>
 		<xacro:insert_visu_LFinger42_link/>
 	</link>
-	<joint name="LFinger42" type="continuous">
+	<joint name="LFinger42" type="fixed">
 		<parent link="LFinger41_link"/>
 		<child link="LFinger42_link"/>
@@ -39,5 +39,5 @@
 		<xacro:insert_visu_RFinger12_link/>
 	</link>
-	<joint name="RFinger12" type="continuous">
+	<joint name="RFinger12" type="fixed">
 		<parent link="RFinger11_link"/>
 		<child link="RFinger12_link"/>
@@ -48,10 +48,10 @@
 	<link name="LFinger33_link">
 		<inertial>
-			<mass value="0"/>
+			<mass value="0.001"/>
 			<inertia ixx="0" ixy="0" ixz="0" iyy="0" iyz="0" izz="0"/>
 		</inertial>
 		<xacro:insert_visu_LFinger33_link/>
 	</link>
-	<joint name="LFinger33" type="continuous">
+	<joint name="LFinger33" type="fixed">
 		<parent link="LFinger32_link"/>
 		<child link="LFinger33_link"/>
@@ -62,10 +62,10 @@
 	<link name="RFinger31_link">
 		<inertial>
-			<mass value="0"/>
+			<mass value="0.001"/>
 			<inertia ixx="0" ixy="0" ixz="0" iyy="0" iyz="0" izz="0"/>
 		</inertial>
 		<xacro:insert_visu_RFinger31_link/>
 	</link>
-	<joint name="RFinger31" type="continuous">
+	<joint name="RFinger31" type="fixed">
 		<parent link="r_wrist"/>
 		<child link="RFinger31_link"/>
@@ -76,10 +76,10 @@
 	<link name="LFinger21_link">
 		<inertial>
-			<mass value="0"/>
+			<mass value="0.001"/>
 			<inertia ixx="0" ixy="0" ixz="0" iyy="0" iyz="0" izz="0"/>
 		</inertial>
 		<xacro:insert_visu_LFinger21_link/>
 	</link>
-	<joint name="LFinger21" type="continuous">
+	<joint name="LFinger21" type="fixed">
 		<parent link="l_wrist"/>
 		<child link="LFinger21_link"/>
@@ -90,10 +90,10 @@
 	<link name="RFinger32_link">
 		<inertial>
-			<mass value="0"/>
+			<mass value="0.001"/>
 			<inertia ixx="0" ixy="0" ixz="0" iyy="0" iyz="0" izz="0"/>
 		</inertial>
 		<xacro:insert_visu_RFinger32_link/>
 	</link>
-	<joint name="RFinger32" type="continuous">
+	<joint name="RFinger32" type="fixed">
 		<parent link="RFinger31_link"/>
 		<child link="RFinger32_link"/>
@@ -109,5 +109,5 @@
 		<xacro:insert_visu_LFinger13_link/>
 	</link>
-	<joint name="LFinger13" type="continuous">
+	<joint name="LFinger13" type="fixed">
 		<parent link="LFinger12_link"/>
 		<child link="LFinger13_link"/>
@@ -118,10 +118,10 @@
 	<link name="LFinger32_link">
 		<inertial>
-			<mass value="0"/>
+			<mass value="0.001"/>
 			<inertia ixx="0" ixy="0" ixz="0" iyy="0" iyz="0" izz="0"/>
 		</inertial>
 		<xacro:insert_visu_LFinger32_link/>
 	</link>
-	<joint name="LFinger32" type="continuous">
+	<joint name="LFinger32" type="fixed">
 		<parent link="LFinger31_link"/>
 		<child link="LFinger32_link"/>
@@ -137,5 +137,5 @@
 		<xacro:insert_visu_LFinger11_link/>
 	</link>
-	<joint name="LFinger11" type="continuous">
+	<joint name="LFinger11" type="fixed">
 		<parent link="l_wrist"/>
 		<child link="LFinger11_link"/>
@@ -146,10 +146,10 @@
 	<link name="RFinger22_link">
 		<inertial>
-			<mass value="0"/>
+			<mass value="0.001"/>
 			<inertia ixx="0" ixy="0" ixz="0" iyy="0" iyz="0" izz="0"/>
 		</inertial>
 		<xacro:insert_visu_RFinger22_link/>
 	</link>
-	<joint name="RFinger22" type="continuous">
+	<joint name="RFinger22" type="fixed">
 		<parent link="RFinger21_link"/>
 		<child link="RFinger22_link"/>
@@ -165,5 +165,5 @@
 		<xacro:insert_visu_RFinger13_link/>
 	</link>
-	<joint name="RFinger13" type="continuous">
+	<joint name="RFinger13" type="fixed">
 		<parent link="RFinger12_link"/>
 		<child link="RFinger13_link"/>
@@ -174,10 +174,10 @@
 	<link name="LFinger22_link">
 		<inertial>
-			<mass value="0"/>
+			<mass value="0.001"/>
 			<inertia ixx="0" ixy="0" ixz="0" iyy="0" iyz="0" izz="0"/>
 		</inertial>
 		<xacro:insert_visu_LFinger22_link/>
 	</link>
-	<joint name="LFinger22" type="continuous">
+	<joint name="LFinger22" type="fixed">
 		<parent link="LFinger21_link"/>
 		<child link="LFinger22_link"/>
@@ -188,10 +188,10 @@
 	<link name="RFinger21_link">
 		<inertial>
-			<mass value="0"/>
+			<mass value="0.001"/>
 			<inertia ixx="0" ixy="0" ixz="0" iyy="0" iyz="0" izz="0"/>
 		</inertial>
 		<xacro:insert_visu_RFinger21_link/>
 	</link>
-	<joint name="RFinger21" type="continuous">
+	<joint name="RFinger21" type="fixed">
 		<parent link="r_wrist"/>
 		<child link="RFinger21_link"/>
@@ -202,10 +202,10 @@
 	<link name="LFinger41_link">
 		<inertial>
-			<mass value="0"/>
+			<mass value="0.001"/>
 			<inertia ixx="0" ixy="0" ixz="0" iyy="0" iyz="0" izz="0"/>
 		</inertial>
 		<xacro:insert_visu_LFinger41_link/>
 	</link>
-	<joint name="LFinger41" type="continuous">
+	<joint name="LFinger41" type="fixed">
 		<parent link="l_wrist"/>
 		<child link="LFinger41_link"/>
@@ -221,5 +221,5 @@
 		<xacro:insert_visu_LFinger12_link/>
 	</link>
-	<joint name="LFinger12" type="continuous">
+	<joint name="LFinger12" type="fixed">
 		<parent link="LFinger11_link"/>
 		<child link="LFinger12_link"/>
@@ -230,10 +230,10 @@
 	<link name="RFinger23_link">
 		<inertial>
-			<mass value="0"/>
+			<mass value="0.001"/>
 			<inertia ixx="0" ixy="0" ixz="0" iyy="0" iyz="0" izz="0"/>
 		</inertial>
 		<xacro:insert_visu_RFinger23_link/>
 	</link>
-	<joint name="RFinger23" type="continuous">
+	<joint name="RFinger23" type="fixed">
 		<parent link="RFinger22_link"/>
 		<child link="RFinger23_link"/>
@@ -249,5 +249,5 @@
 		<xacro:insert_visu_RFinger11_link/>
 	</link>
-	<joint name="RFinger11" type="continuous">
+	<joint name="RFinger11" type="fixed">
 		<parent link="r_wrist"/>
 		<child link="RFinger11_link"/>
@@ -258,10 +258,10 @@
 	<link name="LFinger23_link">
 		<inertial>
-			<mass value="0"/>
+			<mass value="0.001"/>
 			<inertia ixx="0" ixy="0" ixz="0" iyy="0" iyz="0" izz="0"/>
 		</inertial>
 		<xacro:insert_visu_LFinger23_link/>
 	</link>
-	<joint name="LFinger23" type="continuous">
+	<joint name="LFinger23" type="fixed">
 		<parent link="LFinger22_link"/>
 		<child link="LFinger23_link"/>
@@ -272,10 +272,10 @@
 	<link name="LFinger43_link">
 		<inertial>
-			<mass value="0"/>
+			<mass value="0.001"/>
 			<inertia ixx="0" ixy="0" ixz="0" iyy="0" iyz="0" izz="0"/>
 		</inertial>
 		<xacro:insert_visu_LFinger43_link/>
 	</link>
-	<joint name="LFinger43" type="continuous">
+	<joint name="LFinger43" type="fixed">
 		<parent link="LFinger42_link"/>
 		<child link="LFinger43_link"/>
@@ -286,10 +286,10 @@
 	<link name="RFinger43_link">
 		<inertial>
-			<mass value="0"/>
+			<mass value="0.001"/>
 			<inertia ixx="0" ixy="0" ixz="0" iyy="0" iyz="0" izz="0"/>
 		</inertial>
 		<xacro:insert_visu_RFinger43_link/>
 	</link>
-	<joint name="RFinger43" type="continuous">
+	<joint name="RFinger43" type="fixed">
 		<parent link="RFinger42_link"/>
 		<child link="RFinger43_link"/>
@@ -300,10 +300,10 @@
 	<link name="RFinger42_link">
 		<inertial>
-			<mass value="0"/>
+			<mass value="0.001"/>
 			<inertia ixx="0" ixy="0" ixz="0" iyy="0" iyz="0" izz="0"/>
 		</inertial>
 		<xacro:insert_visu_RFinger42_link/>
 	</link>
-	<joint name="RFinger42" type="continuous">
+	<joint name="RFinger42" type="fixed">
 		<parent link="RFinger41_link"/>
 		<child link="RFinger42_link"/>
@@ -314,10 +314,10 @@
 	<link name="LFinger31_link">
 		<inertial>
-			<mass value="0"/>
+			<mass value="0.001"/>
 			<inertia ixx="0" ixy="0" ixz="0" iyy="0" iyz="0" izz="0"/>
 		</inertial>
 		<xacro:insert_visu_LFinger31_link/>
 	</link>
-	<joint name="LFinger31" type="continuous">
+	<joint name="LFinger31" type="fixed">
 		<parent link="l_wrist"/>
 		<child link="LFinger31_link"/>
@@ -328,10 +328,10 @@
 	<link name="RFinger33_link">
 		<inertial>
-			<mass value="0"/>
+			<mass value="0.001"/>
 			<inertia ixx="0" ixy="0" ixz="0" iyy="0" iyz="0" izz="0"/>
 		</inertial>
 		<xacro:insert_visu_RFinger33_link/>
 	</link>
-	<joint name="RFinger33" type="continuous">
+	<joint name="RFinger33" type="fixed">
 		<parent link="RFinger32_link"/>
 		<child link="RFinger33_link"/>
@@ -347,5 +347,5 @@
 		<xacro:insert_visu_LThumb1_link/>
 	</link>
-	<joint name="LThumb1" type="continuous">
+	<joint name="LThumb1" type="fixed">
 		<parent link="l_wrist"/>
 		<child link="LThumb1_link"/>
@@ -361,5 +361,5 @@
 		<xacro:insert_visu_RThumb2_link/>
 	</link>
-	<joint name="RThumb2" type="continuous">
+	<joint name="RThumb2" type="fixed">
 		<parent link="RThumb1_link"/>
 		<child link="RThumb2_link"/>
@@ -375,5 +375,5 @@
 		<xacro:insert_visu_RThumb1_link/>
 	</link>
-	<joint name="RThumb1" type="continuous">
+	<joint name="RThumb1" type="fixed">
 		<parent link="r_wrist"/>
 		<child link="RThumb1_link"/>
@@ -389,5 +389,5 @@
 		<xacro:insert_visu_LThumb2_link/>
 	</link>
-	<joint name="LThumb2" type="continuous">
+	<joint name="LThumb2" type="fixed">
 		<parent link="LThumb1_link"/>
 		<child link="LThumb2_link"/>
