Commit message: configure initial position

File: pepper_description/urdf/pepper1.0_generated_urdf/pepper_arms.xacro (robot description, xacro)
@@ -8,5 +8,5 @@
 		<child link="LShoulder"/>
 		<origin rpy="0 0 0" xyz="-0.057 0.14974 0.08682"/>
-		<axis xyz="0 1.0 0"/>
+		<axis xyz="0 1.0 0" initial_position="1.57" />
 		<limit effort="5.428" lower="-2.08567" upper="2.08567" velocity="7.33998"/>
 	</joint>
@@ -96,5 +96,5 @@
 		<child link="RShoulder"/>
 		<origin rpy="0 0 0" xyz="-0.057 -0.14974 0.08682"/>
-		<axis xyz="0 1.0 0"/>
+		<axis xyz="0 1.0 0" initial_position="1.57" />
 		<limit effort="5.428" lower="-2.08567" upper="2.08567" velocity="7.33998"/>
 	</joint>
